File: ultrablinky.sch (KiCad schematic (older format))
At the start: 120 parts, among them J1 DNP, J2 SJ1-3523N, J3 SJ1-3523N, J4 Barrel_Jack_5.5x2.5, J5 DNP, J6 DNP, J7 Terminal5, J8 SJ1-3523N, Q1 DMP6180SK3Q-13, Q2 DMP6180SK3Q-13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

Commit message: Changed C12 from 50V to 100V
This was changed so that the same 10nF cap could be used in all
locations instead of having two different 10nF parts
Parts:
- C12: Source Mouser 80-C0805C103K5R -> Mouser 80-C0805C103K1R
Changed lines of the file:
@@
 F 2 "Resistor_SMD:R_0805_2012Metric" H 12438 5350 50  0001 C CNN
 F 3 "~" H 12400 5500 50  0001 C CNN
-F 4 "Mouser 80-C0805C103K5R" H 12400 5500 50  0001 C CNN "Source"
+F 4 "Mouser 80-C0805C103K1R" H 12400 5500 50  0001 C CNN "Source"
 	1    12400 5500
 	1    0    0    -1
