File: ultrablinky.sch (KiCad schematic (older format))
At the start: 120 parts, among them J1 DNP, J2 SJ1-3523N, J3 SJ1-3523N, J4 Barrel_Jack_5.5x2.5, J5 DNP, J6 DNP, J7 Terminal5, J8 SJ1-3523N, Q1 DMP6180SK3Q-13, Q2 DMP6180SK3Q-13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

Commit message: Improve rise/fall time
Changed C21 from 10nF to 100pF
Parts:
- C21: value 10nF -> 100pF; Source Mouser 80-C0805C103K1R -> Mouser 80-C0805C101J1G
Changed lines of the file:
@@
 P 4300 6950
 F 0 "C21" H 4150 7050 50  0000 L CNN
-F 1 "10nF" H 4100 6850 50  0000 L CNN
+F 1 "100pF" H 4050 6850 50  0000 L CNN
 F 2 "Capacitor_SMD:C_0805_2012Metric" H 4338 6800 50  0001 C CNN
 F 3 "~" H 4300 6950 50  0001 C CNN
-F 4 "Mouser 80-C0805C103K1R" H 4300 6950 50  0001 C CNN "Source"
+F 4 "Mouser 80-C0805C101J1G" H 4300 6950 50  0001 C CNN "Source"
 	1    4300 6950
 	1    0    0    -1

Commit message: Fixed LED staying on when it shouldn't be
Previously there were two times when the strobe LED stayed on when it
was supposed to be off. First, when the system started, the PWM pin
would float and would not turn off the LED. Secondly, the non-inverting
input of the op amp would not go low enough to completely turn off off
the LED.

The startup problem was fixed by adding a 10k pull-up resistor to the
PWM signal so that it would be high during the time before the code
initialized that signal to be an output and actively drives it.

The second problem was fixed by adding a 22k pull-up to 5V on the
inverting input of the op amp. This kept the inverting input at a higher
voltage and allowed the non-inverting input to completely turn the op
amp output off.
Parts:
- added R44: 22k, Resistor_SMD:R_0805_2012Metric, symbol Device:R
- added R45: 10k, Resistor_SMD:R_0805_2012Metric, symbol Device:R
Connections:
- wire segments 372 -> 379
- no-connect marks 24 -> 23
Other:
- moved on the sheet: C17, R13, R15
Changed lines of the file:
@@
 L power:+5V #PWR0105
 U 1 1 602F5884
-P 3700 6200
-F 0 "#PWR0105" H 3700 6050 50  0001 C CNN
-F 1 "+5V" H 3715 6373 50  0000 C CNN
-F 2 "" H 3700 6200 50  0001 C CNN
-F 3 "" H 3700 6200 50  0001 C CNN
-	1    3700 6200
+P 3700 6050
+F 0 "#PWR0105" H 3700 5900 50  0001 C CNN
+F 1 "+5V" H 3715 6223 50  0000 C CNN
+F 2 "" H 3700 6050 50  0001 C CNN
+F 3 "" H 3700 6050 50  0001 C CNN
+	1    3700 6050
 	1    0    0    -1
 $EndComp
@@
 L power:GND #PWR0112
 U 1 1 60322C1C
-P 4700 3750
-F 0 "#PWR0112" H 4700 3500 50  0001 C CNN
-F 1 "GND" H 4705 3577 50  0000 C CNN
-F 2 "" H 4700 3750 50  0001 C CNN
-F 3 "" H 4700 3750 50  0001 C CNN
-	1    4700 3750
+P 4900 3350
+F 0 "#PWR0112" H 4900 3100 50  0001 C CNN
+F 1 "GND" H 4905 3177 50  0000 C CNN
+F 2 "" H 4900 3350 50  0001 C CNN
+F 3 "" H 4900 3350 50  0001 C CNN
+	1    4900 3350
 	1    0    0    -1
 $EndComp
-Wire Wire Line
-	4700 3750 4700 3350
-Wire Wire Line
-	4700 3350 4600 3350
 $Comp
 L power:GND #PWR0113
@@
 Text Label 2650 7000 0    50   ~ 0
 PWM
-Text Label 5300 3650 0    50   ~ 0
+Text Label 5450 3650 0    50   ~ 0
 PWM
 $Comp
@@
 L Device:R R13
 U 1 1 603080FE
-P 4950 3650
-F 0 "R13" V 4850 3650 50  0000 C CNN
-F 1 "1k" V 4950 3650 50  0000 C CNN
-F 2 "Resistor_SMD:R_0805_2012Metric" V 4880 3650 50  0001 C CNN
-F 3 "~" H 4950 3650 50  0001 C CNN
-F 4 "Mouser 603-RC0805JR-071KL" H 4950 3650 50  0001 C CNN "Source"
-	1    4950 3650
+P 5150 3650
+F 0 "R13" V 5050 3650 50  0000 C CNN
+F 1 "1k" V 5150 3650 50  0000 C CNN
+F 2 "Resistor_SMD:R_0805_2012Metric" V 5080 3650 50  0001 C CNN
+F 3 "~" H 5150 3650 50  0001 C CNN
+F 4 "Mouser 603-RC0805JR-071KL" H 5150 3650 50  0001 C CNN "Source"
+	1    5150 3650
 	0    -1   -1   0
 $EndComp
@@
 	1700 8400 2000 8400
 Wire Wire Line
-	5600 3650 5100 3650
+	5750 3650 5300 3650
 Text Label 1600 6750 0    50   ~ 0
 V1_5
@@
 L power:+5V #PWR0121
 U 1 1 6049CE18
-P 5900 3200
-F 0 "#PWR0121" H 5900 3050 50  0001 C CNN
-F 1 "+5V" H 5900 3400 50  0000 C CNN
-F 2 "" H 5900 3200 50  0001 C CNN
-F 3 "" H 5900 3200 50  0001 C CNN
-	1    5900 3200
+P 6050 3200
+F 0 "#PWR0121" H 6050 3050 50  0001 C CNN
+F 1 "+5V" H 6050 3400 50  0000 C CNN
+F 2 "" H 6050 3200 50  0001 C CNN
+F 3 "" H 6050 3200 50  0001 C CNN
+	1    6050 3200
 	1    0    0    -1
 $EndComp
@@
 	3750 6250 3700 6250
 Wire Wire Line
-	3700 6200 3700 6250
+	3700 6050 3700 6100
 Wire Wire Line
 	4100 6250 4050 6250
@@
 	1    0    0    -1
 $EndComp
-NoConn ~ 4600 3450
 $Comp
 L Device:C C3
@@
 Text Label 1350 3550 0    50   ~ 0
 I2S_LRCLK
-Text Label 5200 3550 0    50   ~ 0
+Text Label 5350 3550 0    50   ~ 0
 I2S_MCLK
 Text Label 1350 1850 0    50   ~ 0
@@
 	1300 3550 1850 3550
 Wire Wire Line
-	4600 3550 4800 3550
+	4600 3550 5000 3550
 $Comp
 L Device:R R?
@@
 L Device:R R15
 U 1 1 609BBB13
-P 4950 3550
-F 0 "R15" V 4850 3550 50  0000 C CNN
-F 1 "33" V 4950 3550 50  0000 C CNN
-F 2 "Resistor_SMD:R_0805_2012Metric" V 4880 3550 50  0001 C CNN
-F 3 "~" H 4950 3550 50  0001 C CNN
-F 4 "Mouser 603-RC0805JR-1333RL" H 4950 3550 50  0001 C CNN "Source"
-	1    4950 3550
+P 5150 3550
+F 0 "R15" V 5050 3550 50  0000 C CNN
+F 1 "33" V 5150 3550 50  0000 C CNN
+F 2 "Resistor_SMD:R_0805_2012Metric" V 5080 3550 50  0001 C CNN
+F 3 "~" H 5150 3550 50  0001 C CNN
+F 4 "Mouser 603-RC0805JR-1333RL" H 5150 3550 50  0001 C CNN "Source"
+	1    5150 3550
 	0    1    1    0
 $EndComp
 Wire Wire Line
-	5100 3550 5600 3550
+	5300 3550 5750 3550
 $Comp
 L Device:R R12
@@
 L Device:C C?
 U 1 1 60601AC5
-P 5900 3400
+P 6050 3400
 AR Path="/5ECF51E5/60601AC5" Ref="C?"  Part="1"
 AR Path="/60601AC5" Ref="C17"  Part="1"
 AR Path="/60675ACD/60601AC5" Ref="C?"  Part="1"
-F 0 "C17" H 6015 3446 50  0000 L CNN
-F 1 "10uF" H 6015 3355 50  0000 L CNN
-F 2 "Capacitor_SMD:C_1206_3216Metric" H 5938 3250 50  0001 C CNN
-F 3 "~" H 5900 3400 50  0001 C CNN
-F 4 "Mouser 187-CL31B106KOHNNWE" H 5900 3400 50  0001 C CNN "Source"
-	1    5900 3400
+F 0 "C17" H 6165 3446 50  0000 L CNN
+F 1 "10uF" H 6165 3355 50  0000 L CNN
+F 2 "Capacitor_SMD:C_1206_3216Metric" H 6088 3250 50  0001 C CNN
+F 3 "~" H 6050 3400 50  0001 C CNN
+F 4 "Mouser 187-CL31B106KOHNNWE" H 6050 3400 50  0001 C CNN "Source"
+	1    6050 3400
 	1    0    0    -1
 $EndComp
 Wire Wire Line
-	4600 3250 5900 3250
+	4600 3250 6050 3250
 $Comp
 L power:GND #PWR0187
 U 1 1 60656145
-P 5900 3550
-F 0 "#PWR0187" H 5900 3300 50  0001 C CNN
-F 1 "GND" H 5905 3377 50  0000 C CNN
-F 2 "" H 5900 3550 50  0001 C CNN
-F 3 "" H 5900 3550 50  0001 C CNN
-	1    5900 3550
+P 6050 3550
+F 0 "#PWR0187" H 6050 3300 50  0001 C CNN
+F 1 "GND" H 6055 3377 50  0000 C CNN
+F 2 "" H 6050 3550 50  0001 C CNN
+F 3 "" H 6050 3550 50  0001 C CNN
+	1    6050 3550
 	1    0    0    -1
 $EndComp
 Wire Wire Line
-	5900 3200 5900 3250
-Connection ~ 5900 3250
+	6050 3200 6050 3250
+Connection ~ 6050 3250
 NoConn ~ 11200 10150
 Wire Wire Line
 	1300 3250 2400 3250
 Wire Wire Line
-	4800 3650 4600 3650
+	5000 3650 4950 3650
 Wire Wire Line
 	1550 8800 1550 8900
@@
 	1    0    0    -1
 $EndComp
+$Comp
+L Device:R R44
+U 1 1 60C5D3B3
+P 3450 6350
+F 0 "R44" V 3350 6350 50  0000 C CNN
+F 1 "22k" V 3450 6350 50  0000 C CNN
+F 2 "Resistor_SMD:R_0805_2012Metric" V 3380 6350 50  0001 C CNN
+F 3 "~" H 3450 6350 50  0001 C CNN
+F 4 "Mouser 603-RC0805JR-0722KL" H 3450 6350 50  0001 C CNN "Source"
+	1    3450 6350
+	-1   0    0    1
+$EndComp
+Wire Wire Line
+	3450 6500 3450 6850
+Connection ~ 3450 6850
+Wire Wire Line
+	3450 6200 3450 6100
+Wire Wire Line
+	3450 6100 3700 6100
+Connection ~ 3700 6100
+Wire Wire Line
+	3700 6100 3700 6250
+$Comp
+L Device:R R45
+U 1 1 60D18074
+P 4800 3800
+F 0 "R45" V 4900 3800 50  0000 C CNN
+F 1 "10k" V 4800 3800 50  0000 C CNN
+F 2 "Resistor_SMD:R_0805_2012Metric" V 4730 3800 50  0001 C CNN
+F 3 "~" H 4800 3800 50  0001 C CNN
+F 4 "Mouser 603-RC0805JR-0710KL" H 4800 3800 50  0001 C CNN "Source"
+	1    4800 3800
+	0    1    1    0
+$EndComp
+Wire Wire Line
+	4600 3350 4900 3350
+Wire Wire Line
+	4600 3450 4650 3450
+Wire Wire Line
+	4650 3450 4650 3800
+Wire Wire Line
+	4950 3800 4950 3650
+Connection ~ 4950 3650
+Wire Wire Line
+	4950 3650 4600 3650
 $EndSCHEMATC

Commit message: Fixed low drive voltage for LED MOSFET
The MC34071ADR2G op amp has a Voh that may be as low as 3.7V when
powered with 5V, which is
not enough to fully turn on the COB LED MOSFET. The power supply was
changed to 36V to allow a much higher voltage.

Also added a 10V zener across the gate and source of the COB LED MOSFET
to avoid having the voltage exceed the maximum Vgs which is 20V.
Parts:
- added D6: BZX84C10LT1G, Diode_SMD:D_SOT-23_ANK, symbol Diode:BZX84Cxx
Connections:
- wire segments 379 -> 381
Other:
- moved on the sheet: D5, HS1, Q7, R43
Changed lines of the file:
@@
 L Transistor_FET:IRLZ44N Q7
 U 1 1 602AB585
-P 5150 6750
-F 0 "Q7" H 5354 6796 50  0000 L CNN
-F 1 "IRFZ44ZPBF" H 5354 6705 50  0000 L CNN
-F 2 "Package_TO_SOT_THT:TO-220-3_Horizontal_TabDown" H 5400 6675 50  0001 L CIN
-F 3 "https://www.infineon.com/dgdl/irfz44zpbf.pdf?fileId=5546d462533600a40153563b6a15221c" H 5150 6750 50  0001 L CNN
-F 4 "Mouser 942-IRFZ44ZPBF, Mouser 534-4724 " H 5150 6750 50  0001 C CNN "Source"
-	1    5150 6750
+P 5350 6750
+F 0 "Q7" H 5554 6796 50  0000 L CNN
+F 1 "IRFZ44ZPBF" H 5554 6705 50  0000 L CNN
+F 2 "Package_TO_SOT_THT:TO-220-3_Horizontal_TabDown" H 5600 6675 50  0001 L CIN
+F 3 "https://www.infineon.com/dgdl/irfz44zpbf.pdf?fileId=5546d462533600a40153563b6a15221c" H 5350 6750 50  0001 L CNN
+F 4 "Mouser 942-IRFZ44ZPBF, Mouser 534-4724 " H 5350 6750 50  0001 C CNN "Source"
+	1    5350 6750
 	1    0    0    -1
 $EndComp
@@
 $EndComp
 Wire Wire Line
-	4950 6750 4700 6750
+	5150 6750 5000 6750
 $Comp
 L Device:C C21
@@
 L Device:R R43
 U 1 1 602AD9D4
-P 5250 7200
-F 0 "R43" H 5320 7246 50  0000 L CNN
-F 1 "0.5 20W" H 5320 7155 50  0000 L CNN
-F 2 "Package_TO_SOT_THT:TO-220-2_Horizontal_TabDown" V 5180 7200 50  0001 C CNN
-F 3 "~" H 5250 7200 50  0001 C CNN
-F 4 "Mouser 652-PWR220T-20-R500F" H 5250 7200 50  0001 C CNN "Source"
-	1    5250 7200
+P 5450 7200
+F 0 "R43" H 5520 7246 50  0000 L CNN
+F 1 "0.5 20W" H 5520 7155 50  0000 L CNN
+F 2 "Package_TO_SOT_THT:TO-220-2_Horizontal_TabDown" V 5380 7200 50  0001 C CNN
+F 3 "~" H 5450 7200 50  0001 C CNN
+F 4 "Mouser 652-PWR220T-20-R500F" H 5450 7200 50  0001 C CNN "Source"
+	1    5450 7200
 	1    0    0    -1
 $EndComp
 Wire Wire Line
-	5250 7350 5250 7400
+	5450 7350 5450 7400
 $Comp
 L power:GND #PWR0101
 U 1 1 602AE939
-P 5250 7400
-F 0 "#PWR0101" H 5250 7150 50  0001 C CNN
-F 1 "GND" H 5255 7227 50  0000 C CNN
-F 2 "" H 5250 7400 50  0001 C CNN
-F 3 "" H 5250 7400 50  0001 C CNN
-	1    5250 7400
+P 5450 7400
+F 0 "#PWR0101" H 5450 7150 50  0001 C CNN
+F 1 "GND" H 5455 7227 50  0000 C CNN
+F 2 "" H 5450 7400 50  0001 C CNN
+F 3 "" H 5450 7400 50  0001 C CNN
+	1    5450 7400
 	1    0    0    -1
 $EndComp
@@
 L Device:LED D5
 U 1 1 602AF7E6
-P 5250 6250
-F 0 "D5" V 5289 6132 50  0000 R CNN
-F 1 "COB LED" V 5198 6132 50  0000 R CNN
-F 2 "0_my_footprints:LED_COB_100W" H 5250 6250 50  0001 C CNN
-F 3 "https://www.amazon.com/gp/product/B01DBZHUXA" H 5250 6250 50  0001 C CNN
-F 4 "Amazon B01DBZHUXA" H 5250 6250 50  0001 C CNN "Source"
-	1    5250 6250
+P 5450 6250
+F 0 "D5" V 5489 6132 50  0000 R CNN
+F 1 "COB LED" V 5398 6132 50  0000 R CNN
+F 2 "0_my_footprints:LED_COB_100W" H 5450 6250 50  0001 C CNN
+F 3 "https://www.amazon.com/gp/product/B01DBZHUXA" H 5450 6250 50  0001 C CNN
+F 4 "Amazon B01DBZHUXA" H 5450 6250 50  0001 C CNN "Source"
+	1    5450 6250
 	0    -1   -1   0
 $EndComp
 Wire Wire Line
-	5250 6400 5250 6550
+	5450 6400 5450 6550
 Wire Notes Line
-	4900 6950 5850 6950
+	5150 6950 6050 6950
 Wire Notes Line
-	5850 6950 5850 6050
+	6050 6950 6050 6050
 Wire Notes Line
-	5850 6050 4900 6050
+	6050 6050 5150 6050
 Wire Notes Line
-	4900 6050 4900 6950
-Text Notes 5450 6150 0    50   ~ 0
+	5150 6050 5150 6950
+Text Notes 5650 6150 0    50   ~ 0
 HEATSINK
 Wire Wire Line
-	5250 6100 5250 6050
-Text Notes 5950 6500 0    50   ~ 0
+	5450 6100 5450 6050
+Text Notes 6150 6500 0    50   ~ 0
 100W LED\nVf = 30V-34V\nIf = 3.5A
 $Comp
@@
 L power:+36V #PWR0102
 U 1 1 602C08DE
-P 5250 6050
-F 0 "#PWR0102" H 5250 5900 50  0001 C CNN
-F 1 "+36V" H 5265 6223 50  0000 C CNN
-F 2 "" H 5250 6050 50  0001 C CNN
-F 3 "" H 5250 6050 50  0001 C CNN
-	1    5250 6050
+P 5450 6050
+F 0 "#PWR0102" H 5450 5900 50  0001 C CNN
+F 1 "+36V" H 5465 6223 50  0000 C CNN
+F 2 "" H 5450 6050 50  0001 C CNN
+F 3 "" H 5450 6050 50  0001 C CNN
+	1    5450 6050
 	1    0    0    -1
 $EndComp
@@
 	1    0    0    -1
 $EndComp
-$Comp
-L power:+5V #PWR0105
-U 1 1 602F5884
-P 3700 6050
-F 0 "#PWR0105" H 3700 5900 50  0001 C CNN
-F 1 "+5V" H 3715 6223 50  0000 C CNN
-F 2 "" H 3700 6050 50  0001 C CNN
-F 3 "" H 3700 6050 50  0001 C CNN
-	1    3700 6050
-	1    0    0    -1
-$EndComp
 Wire Wire Line
 	5700 8900 5700 8950
@@
 	2600 7000 2900 7000
 Wire Wire Line
-	5250 6950 5250 7000
+	5450 6950 5450 7000
 Wire Wire Line
-	4700 7150 5050 7150
+	4700 7150 5000 7150
 Wire Wire Line
-	5050 7150 5050 7000
+	5300 7150 5300 7000
 Wire Wire Line
-	5050 7000 5250 7000
-Connection ~ 5250 7000
+	5300 7000 5450 7000
+Connection ~ 5450 7000
 Wire Wire Line
-	5250 7000 5250 7050
+	5450 7000 5450 7050
 Wire Wire Line
 	2500 6250 2400 6250
@@
 	3750 6250 3700 6250
 Wire Wire Line
-	3700 6050 3700 6100
-Wire Wire Line
 	4100 6250 4050 6250
 Wire Wire Line
@@
 L Mechanical:Heatsink HS1
 U 1 1 6055EC96
-P 6100 6900
-F 0 "HS1" H 6242 7021 50  0000 L CNN
-F 1 "Heatsink" H 6242 6930 50  0000 L CNN
-F 2 "0_my_footprints:Heatsink_70x70mm_ATS-CPX070070025-136-C2-R0" H 6112 6900 50  0001 C CNN
-F 3 "http://www.qats.com/pushPIN/DataSheet/ATS-CPX070070025-136-C2-R0" H 6112 6900 50  0001 C CNN
-F 4 "Mouser 984-CPX07007-136C2R0" H 6100 6900 50  0001 C CNN "Source"
-	1    6100 6900
+P 6300 6900
+F 0 "HS1" H 6442 7021 50  0000 L CNN
+F 1 "Heatsink" H 6442 6930 50  0000 L CNN
+F 2 "0_my_footprints:Heatsink_70x70mm_ATS-CPX070070025-136-C2-R0" H 6312 6900 50  0001 C CNN
+F 3 "http://www.qats.com/pushPIN/DataSheet/ATS-CPX070070025-136-C2-R0" H 6312 6900 50  0001 C CNN
+F 4 "Mouser 984-CPX07007-136C2R0" H 6300 6900 50  0001 C CNN "Source"
+	1    6300 6900
 	1    0    0    -1
 $EndComp
@@
 Wire Wire Line
 	4750 8900 4750 9000
-Text Label 5250 6500 0    50   ~ 0
+Text Label 5450 6500 0    50   ~ 0
 LED_K
-Text Label 4750 7150 0    50   ~ 0
+Text Label 4700 7150 0    50   ~ 0
 ISENSE
 Text Label 1350 3250 0    50   ~ 0
@@
 	3450 6500 3450 6850
 Connection ~ 3450 6850
-Wire Wire Line
-	3450 6200 3450 6100
-Wire Wire Line
-	3450 6100 3700 6100
-Connection ~ 3700 6100
-Wire Wire Line
-	3700 6100 3700 6250
 $Comp
 L Device:R R45
@@
 Wire Wire Line
 	4950 3650 4600 3650
+$Comp
+L Diode:BZX84Cxx D6
+U 1 1 60EC40DE
+P 5000 6950
+F 0 "D6" V 4954 7030 50  0000 L CNN
+F 1 "BZX84C10LT1G" V 5250 6750 50  0000 L CNN
+F 2 "Diode_SMD:D_SOT-23_ANK" H 5000 6775 50  0001 C CNN
+F 3 "https://diotec.com/tl_files/diotec/files/pdf/datasheets/bzx84c2v4.pdf" H 5000 6950 50  0001 C CNN
+F 4 "Mouser 863-BZX84C10LT1G" H 5000 6950 50  0001 C CNN "Source"
+	1    5000 6950
+	0    1    1    0
+$EndComp
+Wire Wire Line
+	5000 7100 5000 7150
+Connection ~ 5000 7150
+Wire Wire Line
+	5000 7150 5300 7150
+Wire Wire Line
+	5000 6800 5000 6750
+Connection ~ 5000 6750
+Wire Wire Line
+	5000 6750 4700 6750
+$Comp
+L power:+5V #PWR01
+U 1 1 60FFEE89
+P 3450 6050
+F 0 "#PWR01" H 3450 5900 50  0001 C CNN
+F 1 "+5V" H 3465 6223 50  0000 C CNN
+F 2 "" H 3450 6050 50  0001 C CNN
+F 3 "" H 3450 6050 50  0001 C CNN
+	1    3450 6050
+	1    0    0    -1
+$EndComp
+Wire Wire Line
+	3450 6050 3450 6200
+Wire Wire Line
+	3700 6050 3700 6250
+$Comp
+L power:+36V #PWR02
+U 1 1 61028729
+P 3700 6050
+F 0 "#PWR02" H 3700 5900 50  0001 C CNN
+F 1 "+36V" H 3715 6223 50  0000 C CNN
+F 2 "" H 3700 6050 50  0001 C CNN
+F 3 "" H 3700 6050 50  0001 C CNN
+	1    3700 6050
+	1    0    0    -1
+$EndComp
 $EndSCHEMATC

Commit message: Increased voltage from 36V to 48V
Previously, the op amp was supplied voltage directly from the 36V power
supply. However, this was not high enough to drive the COB LED to high
currents. Now, the voltage has been increased to 48V, but this
necessitated regulating the voltage to the MC34071A because it cannot
handle 48V.
Parts:
- added Q?: MMBT3904, Package_TO_SOT_SMD:SOT-23, symbol Transistor_BJT:MMBT3904
- added R?: 100k, Resistor_SMD:R_0805_2012Metric, symbol Device:R
Connections:
- net labels added: VDC, VIN, VL, VSW
- net labels removed: +36V, V36IN, V36L, V36SW
- wire segments 381 -> 383
Other:
- note added: "48 VDC\n3A"
- note removed: "36 VDC\n4A"
- moved on the sheet: D6, J6
Changed lines of the file:
@@
 	0    1    1    0
 $EndComp
-Wire Wire Line
-	5150 6750 5000 6750
 $Comp
 L Device:C C21
@@
 	4300 6750 4100 6750
 Connection ~ 4300 6750
-$Comp
-L power:+36V #PWR0102
-U 1 1 602C08DE
-P 5450 6050
-F 0 "#PWR0102" H 5450 5900 50  0001 C CNN
-F 1 "+36V" H 5465 6223 50  0000 C CNN
-F 2 "" H 5450 6050 50  0001 C CNN
-F 3 "" H 5450 6050 50  0001 C CNN
-	1    5450 6050
-	1    0    0    -1
-$EndComp
 Wire Wire Line
 	4300 7150 3450 7150
@@
 	5600 8950 5700 8950
 $Comp
-L power:+36V #PWR0106
-U 1 1 6031BE2D
-P 4550 8400
-F 0 "#PWR0106" H 4550 8250 50  0001 C CNN
-F 1 "+36V" H 4565 8573 50  0000 C CNN
-F 2 "" H 4550 8400 50  0001 C CNN
-F 3 "" H 4550 8400 50  0001 C CNN
-	1    4550 8400
-	1    0    0    -1
-$EndComp
-$Comp
 L Device:D_Schottky D2
 U 1 1 6031F877
@@
 NoConn ~ 2400 2350
 Text Notes 600  8700 0    50   ~ 0
-36 VDC\n4A
+48 VDC\n3A
 Text Notes 8950 8800 0    59   ~ 0
 Photosensitive Epilepsy Warning\n"Between 3-30 hertz (flashes per second) are the common \nrates to trigger seizures but this varies from person to person"\nhttps://epilepsysociety.org.uk/photosensitive-epilepsy
@@
 L Connector_Generic:Conn_01x03 J6
 U 1 1 603BCC4E
-P 1250 4800
-F 0 "J6" H 1300 4500 50  0000 C CNN
-F 1 "DNP" H 1300 4600 50  0000 C CNN
-F 2 "Connector_PinHeader_2.54mm:PinHeader_1x03_P2.54mm_Vertical" H 1250 4800 50  0001 C CNN
-F 3 "~" H 1250 4800 50  0001 C CNN
-F 4 "~" H 1250 4800 50  0001 C CNN "Source"
-	1    1250 4800
+P 800 3450
+F 0 "J6" H 850 3150 50  0000 C CNN
+F 1 "DNP" H 850 3250 50  0000 C CNN
+F 2 "Connector_PinHeader_2.54mm:PinHeader_1x03_P2.54mm_Vertical" H 800 3450 50  0001 C CNN
+F 3 "~" H 800 3450 50  0001 C CNN
+F 4 "~" H 800 3450 50  0001 C CNN "Source"
+	1    800  3450
 	-1   0    0    1
 $EndComp
 Wire Wire Line
-	1450 4900 1550 4900
+	1000 3550 1100 3550
 Wire Wire Line
-	1550 4900 1550 5000
+	1100 3550 1100 3650
 $Comp
 L power:GND #PWR0125
 U 1 1 603E24AC
-P 1550 5000
-F 0 "#PWR0125" H 1550 4750 50  0001 C CNN
-F 1 "GND" H 1555 4827 50  0000 C CNN
-F 2 "" H 1550 5000 50  0001 C CNN
-F 3 "" H 1550 5000 50  0001 C CNN
-	1    1550 5000
+P 1100 3650
+F 0 "#PWR0125" H 1100 3400 50  0001 C CNN
+F 1 "GND" H 1105 3477 50  0000 C CNN
+F 2 "" H 1100 3650 50  0001 C CNN
+F 3 "" H 1100 3650 50  0001 C CNN
+	1    1100 3650
 	1    0    0    -1
 $EndComp
@@
 	5450 6950 5450 7000
 Wire Wire Line
-	4700 7150 5000 7150
-Wire Wire Line
 	5300 7150 5300 7000
 Wire Wire Line
@@
 FOCUS
 Wire Wire Line
-	1300 3350 2400 3350
-Wire Wire Line
-	1300 3450 2400 3450
-Wire Wire Line
 	1300 6650 2000 6650
 Wire Wire Line
@@
 Wire Wire Line
 	2150 3550 2400 3550
-Text Label 1550 4700 0    50   ~ 0
-SDA
-Text Label 1550 4800 0    50   ~ 0
-SCL
-Wire Wire Line
-	1750 4700 1450 4700
-Wire Wire Line
-	1750 4800 1450 4800
 Text Notes 11900 8500 0    50   ~ 0
 I2C\n7-bit addr\n0001010
@@
 	6650 8700 6900 8700
 Text Label 1750 8400 0    50   ~ 0
-V36IN
+VIN
 Text Label 1750 8800 0    50   ~ 0
 GNDIN
 Text Label 2600 8500 0    50   ~ 0
-V36L
+VL
 Connection ~ 4350 8500
 Connection ~ 4750 8500
@@
 	4750 8500 5100 8500
 Text Label 3450 8500 0    50   ~ 0
-V36SW
+VSW
 $Comp
 L Device:C C?
@@
 L Diode:BZX84Cxx D6
 U 1 1 60EC40DE
-P 5000 6950
-F 0 "D6" V 4954 7030 50  0000 L CNN
-F 1 "BZX84C10LT1G" V 5250 6750 50  0000 L CNN
-F 2 "Diode_SMD:D_SOT-23_ANK" H 5000 6775 50  0001 C CNN
-F 3 "https://diotec.com/tl_files/diotec/files/pdf/datasheets/bzx84c2v4.pdf" H 5000 6950 50  0001 C CNN
-F 4 "Mouser 863-BZX84C10LT1G" H 5000 6950 50  0001 C CNN "Source"
-	1    5000 6950
+P 3150 5600
+F 0 "D6" V 3104 5680 50  0000 L CNN
+F 1 "BZX84C10LT1G" V 3150 4950 50  0000 L CNN
+F 2 "Diode_SMD:D_SOT-23_ANK" H 3150 5425 50  0001 C CNN
+F 3 "https://diotec.com/tl_files/diotec/files/pdf/datasheets/bzx84c2v4.pdf" H 3150 5600 50  0001 C CNN
+F 4 "Mouser 863-BZX84C10LT1G" H 3150 5600 50  0001 C CNN "Source"
+	1    3150 5600
 	0    1    1    0
 $EndComp
-Wire Wire Line
-	5000 7100 5000 7150
-Connection ~ 5000 7150
-Wire Wire Line
-	5000 7150 5300 7150
-Wire Wire Line
-	5000 6800 5000 6750
-Connection ~ 5000 6750
-Wire Wire Line
-	5000 6750 4700 6750
 $Comp
 L power:+5V #PWR01
@@
 Wire Wire Line
 	3450 6050 3450 6200
+$Comp
+L power:VDC #PWR?
+U 1 1 6106C1A4
+P 4550 8400
+F 0 "#PWR?" H 4550 8300 50  0001 C CNN
+F 1 "VDC" H 4565 8573 50  0000 C CNN
+F 2 "" H 4550 8400 50  0001 C CNN
+F 3 "" H 4550 8400 50  0001 C CNN
+	1    4550 8400
+	1    0    0    -1
+$EndComp
+$Comp
+L power:VDC #PWR?
+U 1 1 6107AF6A
+P 5450 6050
+F 0 "#PWR?" H 5450 5950 50  0001 C CNN
+F 1 "VDC" H 5465 6223 50  0000 C CNN
+F 2 "" H 5450 6050 50  0001 C CNN
+F 3 "" H 5450 6050 50  0001 C CNN
+	1    5450 6050
+	1    0    0    -1
+$EndComp
+$Comp
+L Transistor_BJT:MMBT3904 Q?
+U 1 1 6108F88A
+P 3600 5350
+F 0 "Q?" H 3791 5396 50  0000 L CNN
+F 1 "MMBT3904" H 3800 5300 50  0000 L CNN
+F 2 "Package_TO_SOT_SMD:SOT-23" H 3800 5275 50  0001 L CIN
+F 3 "http://www.onsemi.com/pdf/datasheet/mmbt3904lt1-d.pdf" H 3600 5350 50  0001 L CNN
+F 4 "Mouser 863-MMBT3904LT3G" H 3600 5350 50  0001 C CNN "Source"
+	1    3600 5350
+	1    0    0    -1
+$EndComp
+Wire Wire Line
+	3700 5550 3700 6250
 Wire Wire Line
-	3700 6050 3700 6250
+	4700 7150 5300 7150
+Wire Wire Line
+	4700 6750 5150 6750
 $Comp
-L power:+36V #PWR02
-U 1 1 61028729
-P 3700 6050
-F 0 "#PWR02" H 3700 5900 50  0001 C CNN
-F 1 "+36V" H 3715 6223 50  0000 C CNN
-F 2 "" H 3700 6050 50  0001 C CNN
-F 3 "" H 3700 6050 50  0001 C CNN
-	1    3700 6050
+L power:GND #PWR?
+U 1 1 610CE73D
+P 3150 5800
+F 0 "#PWR?" H 3150 5550 50  0001 C CNN
+F 1 "GND" H 3155 5627 50  0000 C CNN
+F 2 "" H 3150 5800 50  0001 C CNN
+F 3 "" H 3150 5800 50  0001 C CNN
+	1    3150 5800
 	1    0    0    -1
 $EndComp
+Wire Wire Line
+	3150 5800 3150 5750
+Wire Wire Line
+	3150 5450 3150 5350
+Wire Wire Line
+	3150 5350 3400 5350
+$Comp
+L power:VDC #PWR?
+U 1 1 6114E880
+P 3700 4850
+F 0 "#PWR?" H 3700 4750 50  0001 C CNN
+F 1 "VDC" H 3715 5023 50  0000 C CNN
+F 2 "" H 3700 4850 50  0001 C CNN
+F 3 "" H 3700 4850 50  0001 C CNN
+	1    3700 4850
+	1    0    0    -1
+$EndComp
+Wire Wire Line
+	3700 4850 3700 4900
+$Comp
+L Device:R R?
+U 1 1 6117A498
+P 3150 5150
+F 0 "R?" H 2950 5150 50  0000 L CNN
+F 1 "100k" V 3150 5050 50  0000 L CNN
+F 2 "Resistor_SMD:R_0805_2012Metric" V 3080 5150 50  0001 C CNN
+F 3 "~" H 3150 5150 50  0001 C CNN
+F 4 "Mouser 603-RC0805JR-07100KL" H 3150 5150 50  0001 C CNN "Source"
+	1    3150 5150
+	1    0    0    -1
+$EndComp
+Wire Wire Line
+	3150 5300 3150 5350
+Connection ~ 3150 5350
+Wire Wire Line
+	3150 5000 3150 4900
+Wire Wire Line
+	3150 4900 3700 4900
+Connection ~ 3700 4900
+Wire Wire Line
+	3700 4900 3700 5150
+Wire Wire Line
+	1000 3350 2400 3350
+Wire Wire Line
+	1000 3450 2400 3450
 $EndSCHEMATC
