File: ultrablinky.sch (KiCad schematic (older format))
At the start: 124 parts, among them J1 DNP, J2 SJ1-3523N, J3 SJ1-3523N, J4 Barrel_Jack_5.5x2.5, J5 DNP, J6 SJ1-3523N, J7 Conn_01x05, Q1 DMP6180SK3Q-13, Q2 DMP6180SK3Q-13, Q3 MMBT3904, Q4 MMBT3906, Q5 MMBT3904, Q6 MMBT3904, Q7 IRFZ44ZPBF, SW1 SW_SPDT, SW2 PEC11R-4215F-S0024, SW3 SW_Push, U1 SGTL5000, U2 TPS73618DBV, U3 Teensy4.0, U4 4N25, U5 LM2574HVM-5, U6 MC34071ADR2G, U7 74VHC1G09, U8 DNP, U9 MCP4706A1T-E/CH

Commit message: Changed DAC part to change I2C address
The DAC was changed from MCP4706A1 to MCP4706A0. This is the same
functionality, but the I2C address was changed from 1100001 to 1100000.
This part seems to have somewhat better availability.
Parts:
- U9: value MCP4706A1T-E/CH -> MCP4706A0T-E/CH; Source Mouser 579-MCP4706A1TECH -> Mouser 579-MCP4706A0TECH
Other:
- note added: "I2C\n7-bit addr\n1100000"
- note removed: "I2C\n7-bit addr\n1100001"
Changed lines of the file:
@@
 P 2200 6300
 F 0 "U9" H 1800 6700 50  0000 L CNN
-F 1 "MCP4706A1T-E/CH" H 1400 6600 50  0000 L CNN
+F 1 "MCP4706A0T-E/CH" H 1400 6600 50  0000 L CNN
 F 2 "Package_TO_SOT_SMD:SOT-23-6" H 2200 6050 50  0001 C CNN
 F 3 "" H 2200 6300 50  0001 C CNN
-F 4 "Mouser 579-MCP4706A1TECH" H 2200 6300 50  0001 C CNN "Source"
+F 4 "Mouser 579-MCP4706A0TECH" H 2200 6300 50  0001 C CNN "Source"
 	1    2200 6300
 	1    0    0    -1
@@
 $EndComp
 Text Notes 1750 6750 0    50   ~ 0
-I2C\n7-bit addr\n1100001
+I2C\n7-bit addr\n1100000
 $Comp
 L Device:C C15
